Commit message: added moveit group interfcae nodes

File: xarm_description/urdf/xarm7.urdf (robot description, URDF)
Before this commit: robot UF_ROBOT, 10 links, 9 joints
Links:
- added link left_finger, mass 0.048304; collision mesh filename=package://xarm_description/meshes/gripper/xarm/left_finger.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; visual mesh filename=package://xarm_description/meshes/gripper/xarm/left_finger.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
- added link left_inner_knuckle, mass 0.0230125781256706; collision mesh filename=package://xarm_description/meshes/gripper/xarm/left_inner_k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; visual mesh filename=package://xarm_description/meshes/gripper/xarm/left_inner_k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
- added link left_outer_knuckle, mass 0.033618; collision mesh filename=package://xarm_description/meshes/gripper/xarm/left_outer_k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; visual mesh filename=package://xarm_description/meshes/gripper/xarm/left_outer_k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
- added link link_tcp
- added link right_finger, mass 0.048304; collision mesh filename=package://xarm_description/meshes/gripper/xarm/right_finger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; visual mesh filename=package://xarm_description/meshes/gripper/xarm/right_finger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
- added link right_inner_knuckle, mass 0.023013; collision mesh filename=package://xarm_description/meshes/gripper/xarm/right_inner_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; visual mesh filename=package://xarm_description/meshes/gripper/xarm/right_inner_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
- added link right_outer_knuckle, mass 0.033618; collision mesh filename=package://xarm_description/meshes/gripper/xarm/right_outer_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; visual mesh filename=package://xarm_description/meshes/gripper/xarm/right_outer_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
- added link xarm_gripper_base_link, mass 0.54156; collision mesh filename=package://xarm_description/meshes/gripper/xarm/base_link.stl; visual mesh filename=package://xarm_description/meshes/gripper/xarm/base_link.stl
Joints:
- added joint drive_joint: type revolute, parent xarm_gripper_base_link, child left_outer_knuckle, origin xyz=0 0.035 0.059098 rpy=0 0 0, axis 1 0 0, limit lower=0 upper=0.85 effort=50 velocity=2
- added joint gripper_fix: type fixed, parent link_eef, child xarm_gripper_base_link, origin xyz=0 0 0 rpy=0 0 0
- added joint joint_tcp: type fixed, parent xarm_gripper_base_link, child link_tcp, origin xyz=0 0 0.172 rpy=0 0 0
- added joint left_finger_joint: type revolute, parent left_outer_knuckle, child left_finger, origin xyz=0 0.035465 0.042039 rpy=0 0 0, axis -1 0 0, limit lower=0 upper=0.85 effort=50 velocity=2, mimic joint=drive_joint multiplier=1 offset=0
- added joint left_inner_knuckle_joint: type revolute, parent xarm_gripper_base_link, child left_inner_knuckle, origin xyz=0 0.02 0.074098 rpy=0 0 0, axis 1 0 0, limit lower=0 upper=0.85 effort=50 velocity=2, mimic joint=drive_joint multiplier=1 offset=0
- added joint right_finger_joint: type revolute, parent right_outer_knuckle, child right_finger, origin xyz=0 -0.035465 0.042039 rpy=0 0 0, axis 1 0 0, limit lower=0 upper=0.85 effort=50 velocity=2, mimic joint=drive_joint multiplier=1 offset=0
- added joint right_inner_knuckle_joint: type revolute, parent xarm_gripper_base_link, child right_inner_knuckle, origin xyz=0 -0.02 0.074098 rpy=0 0 0, axis -1 0 0, limit lower=0 upper=0.85 effort=50 velocity=2, mimic joint=drive_joint multiplier=1 offset=0
- added joint right_outer_knuckle_joint: type revolute, parent xarm_gripper_base_link, child right_outer_knuckle, origin xyz=0 -0.035 0.059098 rpy=0 0 0, axis -1 0 0, limit lower=0 upper=0.85 effort=50 velocity=2, mimic joint=drive_joint multiplier=1 offset=0
- joint joint7: origin xyz=0.076 0.097 0 rpy=-1.5708 0 0 -> xyz=0.097 -0.076 0 rpy=1.5708 0 1.5708

File: xarm_description/urdf/xarm_device.urdf.xacro (robot description, xacro)
@@ -6,5 +6,5 @@
   <xacro:arg name="effort_control" default="false"/>
   <xacro:arg name="velocity_control" default="false"/>
-  <xacro:arg name="add_gripper" default="false"/>
+  <xacro:arg name="add_gripper" default="true"/>
   <xacro:arg name="add_vacuum_gripper" default="false"/>
   <xacro:arg name="model1300" default="false"/>

File: xarm_moveit_config/srdf/_xarm7_macro.srdf.xacro (robot description, xacro)
@@ -1,3 +1,3 @@
-<?xml version="1.0.0" ?>
+<?xml version="1.0" ?>
 <!-- This does not replace URDF, and is not an extension of URDF.
   This is a format for representing semantic information about the robot structure.
