Commit message: added node to plan and execute trajectory for home to A then B then C

File: xarm_description/urdf/gripper/xarm_gripper.urdf.xacro (robot description, xacro)
@@ -182,5 +182,19 @@
       <mimic joint="${prefix}drive_joint" multiplier="1" offset="0" />
     </joint>
-    <link name="${prefix}link_tcp" />
+    <link name="${prefix}link_tcp">
+      <visual>
+        <origin xyz = "0 0 0" rpy = "0 0 0"/>
+        <material name="blue"/>
+        <geometry>
+          <sphere radius = "0.01"/>
+        </geometry>
+      </visual>
+      <collision>
+        <origin xyz = "0 0 0" rpy = "0 0 0"/>
+        <geometry>
+          <sphere radius = "0.01"/>
+        </geometry>
+      </collision>
+    </link>
     <joint name="${prefix}joint_tcp" type="fixed">
       <origin xyz="0 0 0.172" rpy="0 0 0" />

Commit message: Added tcp pose publisher

File: xarm_description/urdf/gripper/xarm_gripper.urdf.xacro (robot description, xacro)
@@ -183,5 +183,5 @@
     </joint>
     <link name="${prefix}link_tcp">
-      <visual>
+      <!-- <visual>
         <origin xyz = "0 0 0" rpy = "0 0 0"/>
         <material name="blue"/>
@@ -195,5 +195,5 @@
           <sphere radius = "0.01"/>
         </geometry>
-      </collision>
+      </collision> -->
     </link>
     <joint name="${prefix}joint_tcp" type="fixed">
