Commit message: matched home pose of gripper and the table in gazebo to match the workstation

File: xarm_description/urdf/xarm7/xarm7.urdf.xacro (robot description, xacro)
@@ -194,17 +194,17 @@
       <xacro:common_link_inertial
         link_inertial_params="${inertial_params['link6']}"
-        origin_rpy="0 0 0"/>
+        origin_rpy="0 0 -1.5708"/>
       <xacro:common_link_visual
         mesh_filename="xarm7/visual/link6"
         origin_xyz="0 0 0"
-        origin_rpy="0 0 0"
+        origin_rpy="0 0 -1.5708"
         material_name="${prefix}White" />
       <xacro:common_link_collision
         mesh_filename="xarm7/visual/link6"
         origin_xyz="0 0 0"
-        origin_rpy="0 0 0" />
+        origin_rpy="0 0 -1.5708" />
     </link>
     <joint name="${prefix}joint6" type="revolute">
-      <!-- <origin xyz="0 0 0" rpy="1.5708 0 0" /> -->
+      <origin xyz="0 0 0" rpy="1.5708 0 0" />
       <xacro:common_joint_origin joint_kinematic_params="${kinematics_params['joint6']}" />
       <parent link="${prefix}link5" />
@@ -221,5 +221,5 @@
       <xacro:common_link_inertial
         link_inertial_params="${inertial_params['link7']}"
-        origin_rpy="0 0 0"/>
+        origin_rpy="0 0 0" />
       <xacro:common_link_visual
         mesh_filename="${end_tool_visual_filename}"
@@ -233,5 +233,5 @@
     </link>
     <joint name="${prefix}joint7" type="revolute">
-      <!-- <origin xyz="0.076 0.097 0" rpy="-1.5708 0 0" /> -->
+      <origin xyz="0.097 -0.076 0" rpy="1.5708 0 1.5708" />
       <xacro:common_joint_origin joint_kinematic_params="${kinematics_params['joint7']}" />
       <parent link="${prefix}link6" />

Commit message: edited joint angles

File: xarm_description/urdf/xarm7/xarm7.urdf.xacro (robot description, xacro)
@@ -233,4 +233,5 @@
     </link>
     <joint name="${prefix}joint7" type="revolute">
+      <!-- <origin xyz="0.097 -0.076 0" rpy="1.5708 0 1.5708" /> -->
       <origin xyz="0.097 -0.076 0" rpy="1.5708 0 1.5708" />
       <xacro:common_joint_origin joint_kinematic_params="${kinematics_params['joint7']}" />

Commit message: reverted pose of gripper in urdf

File: xarm_description/urdf/xarm7/xarm7.urdf.xacro (robot description, xacro)
@@ -194,14 +194,14 @@
       <xacro:common_link_inertial
         link_inertial_params="${inertial_params['link6']}"
-        origin_rpy="0 0 -1.5708"/>
+        origin_rpy="0 0 0"/>
       <xacro:common_link_visual
         mesh_filename="xarm7/visual/link6"
         origin_xyz="0 0 0"
-        origin_rpy="0 0 -1.5708"
+        origin_rpy="0 0 0"
         material_name="${prefix}White" />
       <xacro:common_link_collision
         mesh_filename="xarm7/visual/link6"
         origin_xyz="0 0 0"
-        origin_rpy="0 0 -1.5708" />
+        origin_rpy="0 0 0" />
     </link>
     <joint name="${prefix}joint6" type="revolute">
@@ -234,5 +234,5 @@
     <joint name="${prefix}joint7" type="revolute">
       <!-- <origin xyz="0.097 -0.076 0" rpy="1.5708 0 1.5708" /> -->
-      <origin xyz="0.097 -0.076 0" rpy="1.5708 0 1.5708" />
+      <!-- <origin xyz="0.097 -0.076 0" rpy="1.5708 0 1.5708" />  -->
       <xacro:common_joint_origin joint_kinematic_params="${kinematics_params['joint7']}" />
       <parent link="${prefix}link6" />

File: xarm_moveit_config/srdf/_xarm7_macro.srdf.xacro (robot description, xacro)
@@ -42,5 +42,5 @@
       <joint name="${prefix}joint4" value="0.0" />
       <joint name="${prefix}joint5" value="0.0" />
-      <joint name="${prefix}joint6" value="0.0" />
+           <joint name="${prefix}joint6" value="-1.5708" />
       <joint name="${prefix}joint7" value="0.0" />
     </group_state>
@@ -51,5 +51,5 @@
       <joint name="${prefix}joint4" value="0.0" />
       <joint name="${prefix}joint5" value="0.0" />
-      <joint name="${prefix}joint6" value="0.0" />
+           <joint name="${prefix}joint6" value="-1.5708" />
       <joint name="${prefix}joint7" value="0.0" />
     </group_state>
@@ -60,5 +60,5 @@
       <joint name="${prefix}joint4" value="0.0" />
       <joint name="${prefix}joint5" value="0.0" />
-      <joint name="${prefix}joint6" value="0.0" />
+           <joint name="${prefix}joint6" value="-1.5708" />
       <joint name="${prefix}joint7" value="0.0" />
     </group_state>
@@ -69,5 +69,5 @@
       <joint name="${prefix}joint4" value="0.0" />
       <joint name="${prefix}joint5" value="-1.5708" />
-      <joint name="${prefix}joint6" value="0.0" />
+           <joint name="${prefix}joint6" value="-1.5708" />
       <joint name="${prefix}joint7" value="0.0" />
     </group_state>

Commit message: reverted robot's pose to the default pose as in the master repo

File: xarm_description/urdf/xarm7/xarm7.urdf.xacro (robot description, xacro)
@@ -233,6 +233,6 @@
     </link>
     <joint name="${prefix}joint7" type="revolute">
+      <!-- <origin xyz="0.076 0.097 0" rpy="-1.5708 0 0" /> -->
       <!-- <origin xyz="0.097 -0.076 0" rpy="1.5708 0 1.5708" /> -->
-      <!-- <origin xyz="0.097 -0.076 0" rpy="1.5708 0 1.5708" />  -->
       <xacro:common_joint_origin joint_kinematic_params="${kinematics_params['joint7']}" />
       <parent link="${prefix}link6" />

Commit message: similar pose as real arm

File: xarm_description/urdf/xarm7/xarm7.urdf.xacro (robot description, xacro)
@@ -206,5 +206,5 @@
     </link>
     <joint name="${prefix}joint6" type="revolute">
-      <origin xyz="0 0 0" rpy="1.5708 0 0" />
+      <!-- <origin xyz="0 0 0" rpy="1.5708 0 0" /> -->
       <xacro:common_joint_origin joint_kinematic_params="${kinematics_params['joint6']}" />
       <parent link="${prefix}link5" />

Commit message: Defined joint6 yaw value based on whether on simulation or hardware

File: xarm_description/urdf/xarm7/xarm7.urdf.xacro (robot description, xacro)
@@ -1,15 +1,5 @@
 <?xml version="1.0"?>
 <robot xmlns:xacro="http://ros.org/wiki/xacro">
-  <xacro:macro name="xarm7_urdf" params="prefix
-    joint1_lower_limit:=${-2.0*pi}  joint1_upper_limit:=${2.0*pi}
-    joint2_lower_limit:=${-2.059}  joint2_upper_limit:=${2.0944}
-    joint3_lower_limit:=${-2.0*pi}  joint3_upper_limit:=${2.0*pi}
-    joint4_lower_limit:=${-0.19198}  joint4_upper_limit:=${3.927}
-    joint5_lower_limit:=${-2.0*pi}  joint5_upper_limit:=${2.0*pi}
-    joint6_lower_limit:=${-1.69297}  joint6_upper_limit:=${pi}
-    joint7_lower_limit:=${-2.0*pi}  joint7_upper_limit:=${2.0*pi}
-    model1300:=false
-    inertial_params_filename:='' kinematics_params_filename:='' "
-    >
+  <xacro:macro name="xarm7_urdf" params="prefix joint1_lower_limit:=${-2.0*pi} joint1_upper_limit:=${2.0*pi} joint2_lower_limit:=${-2.059} joint2_upper_limit:=${2.0944} joint3_lower_limit:=${-2.0*pi} joint3_upper_limit:=${2.0*pi} joint4_lower_limit:=${-0.19198} joint4_upper_limit:=${3.927} joint5_lower_limit:=${-2.0*pi} joint5_upper_limit:=${2.0*pi} joint6_lower_limit:=${-1.69297} joint6_upper_limit:=${pi} joint7_lower_limit:=${-2.0*pi} joint7_upper_limit:=${2.0*pi} model1300:=false inertial_params_filename:='' kinematics_params_filename:='' ">
     <!-- define property -->
     <xacro:if value="${model1300}">
@@ -42,31 +32,13 @@
         <origin xyz="-0.021131 -0.0016302 0.056488" rpy="0 0 0" />
         <mass value="0.88556" />
-        <inertia
-          ixx="0.0030595" ixy="0.00012259" ixz="-0.00062705"
-          iyy="0.0037783" iyz="0.00027023" izz="0.0020125" />
+        <inertia ixx="0.0030595" ixy="0.00012259" ixz="-0.00062705" iyy="0.0037783" iyz="0.00027023" izz="0.0020125" />
       </inertial>
-      <xacro:common_link_visual
-        mesh_filename="xarm7/visual/link_base"
-        origin_xyz="0 0 0"
-        origin_rpy="0 0 0"
-        material_name="${prefix}White" />
-      <xacro:common_link_collision
-        mesh_filename="xarm7/visual/link_base"
-        origin_xyz="0 0 0"
-        origin_rpy="0 0 0" />
+      <xacro:common_link_visual mesh_filename="xarm7/visual/link_base" origin_xyz="0 0 0" origin_rpy="0 0 0" material_name="${prefix}White" />
+      <xacro:common_link_collision mesh_filename="xarm7/visual/link_base" origin_xyz="0 0 0" origin_rpy="0 0 0" />
     </link>
     <link name="${prefix}link1">
-      <xacro:common_link_inertial
-        link_inertial_params="${inertial_params['link1']}"
-        origin_rpy="0 0 0"/>
-      <xacro:common_link_visual
-        mesh_filename="xarm7/visual/link1"
-        origin_xyz="0 0 0"
-        origin_rpy="0 0 0"
-        material_name="${prefix}White" />
-      <xacro:common_link_collision
-        mesh_filename="xarm7/visual/link1"
-        origin_xyz="0 0 0"
-        origin_rpy="0 0 0" />
+      <xacro:common_link_inertial link_inertial_params="${inertial_params['link1']}" origin_rpy="0 0 0"/>
+      <xacro:common_link_visual mesh_filename="xarm7/visual/link1" origin_xyz="0 0 0" origin_rpy="0 0 0" material_name="${prefix}White" />
+      <xacro:common_link_collision mesh_filename="xarm7/visual/link1" origin_xyz="0 0 0" origin_rpy="0 0 0" />
     </link>
     <joint name="${prefix}joint1" type="revolute">
@@ -76,24 +48,11 @@
       <child link="${prefix}link1" />
       <axis xyz="0 0 1" />
-      <limit
-        lower="${joint1_lower_limit}"
-        upper="${joint1_upper_limit}"
-        effort="50"
-        velocity="3.14" />
+      <limit lower="${joint1_lower_limit}" upper="${joint1_upper_limit}" effort="50" velocity="3.14" />
       <dynamics damping="10" friction="1" />
     </joint>
     <link name="${prefix}link2">
-      <xacro:common_link_inertial
-        link_inertial_params="${inertial_params['link2']}"
-        origin_rpy="0 0 0"/>
-      <xacro:common_link_visual
-        mesh_filename="xarm7/visual/link2"
-        origin_xyz="0 0 0"
-        origin_rpy="0 0 0"
-        material_name="${prefix}White" />
-      <xacro:common_link_collision
-        mesh_filename="xarm7/visual/link2"
-        origin_xyz="0 0 0"
-        origin_rpy="0 0 0" />
+      <xacro:common_link_inertial link_inertial_params="${inertial_params['link2']}" origin_rpy="0 0 0"/>
+      <xacro:common_link_visual mesh_filename="xarm7/visual/link2" origin_xyz="0 0 0" origin_rpy="0 0 0" material_name="${prefix}White" />
+      <xacro:common_link_collision mesh_filename="xarm7/visual/link2" origin_xyz="0 0 0" origin_rpy="0 0 0" />
     </link>
     <joint name="${prefix}joint2" type="revolute">
@@ -103,24 +62,11 @@
       <child link="${prefix}link2" />
       <axis xyz="0 0 1" />
-      <limit
-        lower="${joint2_lower_limit}"
-        upper="${joint2_upper_limit}"
-        effort="50"
-        velocity="3.14" />
+      <limit lower="${joint2_lower_limit}" upper="${joint2_upper_limit}" effort="50" velocity="3.14" />
       <dynamics damping="10" friction="1" />
     </joint>
     <link name="${prefix}link3">
-      <xacro:common_link_inertial
-        link_inertial_params="${inertial_params['link3']}"
-        origin_rpy="0 0 0"/>
-      <xacro:common_link_visual
-        mesh_filename="xarm7/visual/link3"
-        origin_xyz="0 0 0"
-        origin_rpy="0 0 0"
-        material_name="${prefix}White" />
-      <xacro:common_link_collision
-        mesh_filename="xarm7/visual/link3"
-        origin_xyz="0 0 0"
-        origin_rpy="0 0 0" />
+      <xacro:common_link_inertial link_inertial_params="${inertial_params['link3']}" origin_rpy="0 0 0"/>
+      <xacro:common_link_visual mesh_filename="xarm7/visual/link3" origin_xyz="0 0 0" origin_rpy="0 0 0" material_name="${prefix}White" />
+      <xacro:common_link_collision mesh_filename="xarm7/visual/link3" origin_xyz="0 0 0" origin_rpy="0 0 0" />
     </link>
     <joint name="${prefix}joint3" type="revolute">
@@ -130,24 +76,11 @@
       <child link="${prefix}link3" />
       <axis xyz="0 0 1" />
-      <limit
-        lower="${joint3_lower_limit}"
-        upper="${joint3_upper_limit}"
-        effort="30"
-        velocity="3.14" />
+      <limit lower="${joint3_lower_limit}" upper="${joint3_upper_limit}" effort="30" velocity="3.14" />
       <dynamics damping="5" friction="1" />
     </joint>
     <link name="${prefix}link4">
-      <xacro:common_link_inertial
-        link_inertial_params="${inertial_params['link4']}"
-        origin_rpy="0 0 0"/>
-      <xacro:common_link_visual
-        mesh_filename="xarm7/visual/link4"
-        origin_xyz="0 0 0"
-        origin_rpy="0 0 0"
-        material_name="${prefix}White" />
-      <xacro:common_link_collision
-        mesh_filename="xarm7/visual/link4"
-        origin_xyz="0 0 0"
-        origin_rpy="0 0 0" />
+      <xacro:common_link_inertial link_inertial_params="${inertial_params['link4']}" origin_rpy="0 0 0"/>
+      <xacro:common_link_visual mesh_filename="xarm7/visual/link4" origin_xyz="0 0 0" origin_rpy="0 0 0" material_name="${prefix}White" />
+      <xacro:common_link_collision mesh_filename="xarm7/visual/link4" origin_xyz="0 0 0" origin_rpy="0 0 0" />
     </link>
     <joint name="${prefix}joint4" type="revolute">
@@ -157,24 +90,11 @@
       <child link="${prefix}link4" />
       <axis xyz="0 0 1" />
-      <limit
-        lower="${joint4_lower_limit}"
-        upper="${joint4_upper_limit}"
-        effort="30"
-        velocity="3.14" />
+      <limit lower="${joint4_lower_limit}" upper="${joint4_upper_limit}" effort="30" velocity="3.14" />
       <dynamics damping="5" friction="1" />
     </joint>
     <link name="${prefix}link5">
-      <xacro:common_link_inertial
-        link_inertial_params="${inertial_params['link5']}"
-        origin_rpy="0 0 0"/>
-      <xacro:common_link_visual
-        mesh_filename="xarm7/visual/link5"
-        origin_xyz="0 0 0"
-        origin_rpy="0 0 0"
-        material_name="${prefix}White" />
-      <xacro:common_link_collision
-        mesh_filename="xarm7/visual/link5"
-        origin_xyz="0 0 0"
-        origin_rpy="0 0 0" />
+      <xacro:common_link_inertial link_inertial_params="${inertial_params['link5']}" origin_rpy="0 0 0"/>
+      <xacro:common_link_visual mesh_filename="xarm7/visual/link5" origin_xyz="0 0 0" origin_rpy="0 0 0" material_name="${prefix}White" />
+      <xacro:common_link_collision mesh_filename="xarm7/visual/link5" origin_xyz="0 0 0" origin_rpy="0 0 0" />
     </link>
     <joint name="${prefix}joint5" type="revolute">
@@ -184,51 +104,32 @@
       <child link="${prefix}link5" />
       <axis xyz="0 0 1" />
-      <limit
-        lower="${joint5_lower_limit}"
-        upper="${joint5_upper_limit}"
-        effort="30"
-        velocity="3.14" />
+      <limit lower="${joint5_lower_limit}" upper="${joint5_upper_limit}" effort="30" velocity="3.14" />
       <dynamics damping="5" friction="1" />
     </joint>
     <link name="${prefix}link6">
-      <xacro:common_link_inertial
-        link_inertial_params="${inertial_params['link6']}"
-        origin_rpy="0 0 0"/>
-      <xacro:common_link_visual
-        mesh_filename="xarm7/visual/link6"
-        origin_xyz="0 0 0"
-        origin_rpy="0 0 0"
-        material_name="${prefix}White" />
-      <xacro:common_link_collision
-        mesh_filename="xarm7/visual/link6"
-        origin_xyz="0 0 0"
-        origin_rpy="0 0 0" />
+      <xacro:common_link_inertial link_inertial_params="${inertial_params['link6']}" origin_rpy="0 0 0"/>
+      <xacro:common_link_visual mesh_filename="xarm7/visual/link6" origin_xyz="0 0 0" origin_rpy="0 0 0" material_name="${prefix}White" />
+      <xacro:common_link_collision mesh_filename="xarm7/visual/link6" origin_xyz="0 0 0" origin_rpy="0 0 0" />
     </link>
     <joint name="${prefix}joint6" type="revolute">
-      <!-- <origin xyz="0 0 0" rpy="1.5708 0 0" /> -->
-      <xacro:common_joint_origin joint_kinematic_params="${kinematics_params['joint6']}" />
+      <!-- If on hardware yaw = 0 -->
+      <xacro:if value = "${robot_ip == '192.1.168.225'}">
+        <!-- <origin xyz="0 0 0" rpy="1.5708 0 0" /> -->
+        <xacro:common_joint_origin joint_kinematic_params="${kinematics_params['joint6']}" />
+      </xacro:if>
+      <!-- if on simulation yaw = 1.5706 -->
+      <xacro:unless value = "${robot_ip == '192.1.168.225'}">
+        <origin xyz="0 0 0" rpy="1.5708 1.5708 0" />
+      </xacro:unless>
       <parent link="${prefix}link5" />
       <child link="${prefix}link6" />
       <axis xyz="0 0 1" />
-      <limit
-        lower="${joint6_lower_limit}"
-        upper="${joint6_upper_limit}"
-        effort="20"
-        velocity="3.14" />
+      <limit lower="${joint6_lower_limit}" upper="${joint6_upper_limit}" effort="20" velocity="3.14" />
       <dynamics damping="2" friction="1" />
     </joint>
     <link name="${prefix}link7">
-      <xacro:common_link_inertial
-        link_inertial_params="${inertial_params['link7']}"
-        origin_rpy="0 0 0" />
-      <xacro:common_link_visual
-        mesh_filename="${end_tool_visual_filename}"
-        origin_xyz="0 0 0"
-        origin_rpy="0 0 0"
-        material_name="${prefix}Silver" />
-      <xacro:common_link_collision
-        mesh_filename="${end_tool_collision_filename}"
-        origin_xyz="0 0 0"
-        origin_rpy="0 0 0" />
+      <xacro:common_link_inertial link_inertial_params="${inertial_params['link7']}" origin_rpy="0 0 0" />
+      <xacro:common_link_visual mesh_filename="${end_tool_visual_filename}" origin_xyz="0 0 0" origin_rpy="0 0 0" material_name="${prefix}Silver" />
+      <xacro:common_link_collision mesh_filename="${end_tool_collision_filename}" origin_xyz="0 0 0" origin_rpy="0 0 0" />
     </link>
     <joint name="${prefix}joint7" type="revolute">
@@ -239,9 +140,5 @@
       <child link="${prefix}link7" />
       <axis xyz="0 0 1" />
-      <limit
-        lower="${joint7_lower_limit}"
-        upper="${joint7_upper_limit}"
-        effort="20"
-        velocity="3.14" />
+      <limit lower="${joint7_lower_limit}" upper="${joint7_upper_limit}" effort="20" velocity="3.14" />
       <dynamics damping="2" friction="1" />
     </joint>

Commit message: added table plane

File: xarm_description/urdf/xarm7/xarm7.urdf.xacro (robot description, xacro)
@@ -28,4 +28,28 @@
     </xacro:unless>
     <xacro:property name="kinematics_params" value="${kinematics_config['kinematics']}"/>
+    <!-- Table plane to assist in collision detection and thus in trajectory generation  -->
+    <link name="${prefix}table_plane">
+      <visual>
+        <origin xyz="0.0 0.0 0.0" rpy="0.0 0.0 0.0"/>
+        <geometry>
+          <mesh filename="package://xarm_description/meshes/xarm7/visual/table_plane.stl" scale="0.0001 0.0001 0.0005"/>
+          <material name="Wood">
+            <color rgba="0.219 0.445 0.286 1.0"/>
+          <texture filename=""/>
+        </material>
+        </geometry>
+      </visual>
+      <collision>
+        <origin xyz="0.0 0.0 0.0" rpy="0.0 0.0 0.0"/>
+        <geometry>
+          <mesh filename="package://xarm_description/meshes/xarm7/visual/table_plane.stl" scale="0.0001 0.0001 0.0005"/>
+        </geometry>
+      </collision>
+    </link>
+    <joint name="${prefix}link_base_table_plane_joint" type="fixed">
+      <origin xyz="0.6 -0.6 -0.02" rpy="0.0 0.0 1.5708"/>
+      <parent link="world"/>
+      <child link="${prefix}table_plane"/>
+    </joint>
     <link name="${prefix}link_base">
       <inertial>

File: xarm_description/urdf/xarm_device_macro.xacro (robot description, xacro)
@@ -70,4 +70,5 @@
       <parent link="${attach_to}" />
       <child link="${prefix}link_base" />
+      <!-- <child link="${prefix}table_plane"/> -->
       <origin xyz="${attach_xyz}" rpy="${attach_rpy}" />
     </joint>
