Commit message: updated how_to_run file

File: xarm_description/urdf/xarm7/xarm7.urdf.xacro (robot description, xacro)
@@ -144,5 +144,6 @@
       <!-- if on simulation yaw = 1.5706 -->
       <xacro:unless value = "${robot_ip == '192.1.168.225'}">
-        <origin xyz="0 0 0" rpy="1.5708 1.5708 0" />
+        <!-- <origin xyz="0 0 0" rpy="1.5708 1.5708 0" /> -->
+        <xacro:common_joint_origin joint_kinematic_params="${kinematics_params['joint6']}" />
       </xacro:unless>
       <parent link="${prefix}link5" />

File: xarm_moveit_config/srdf/_xarm7_macro.srdf.xacro (robot description, xacro)
@@ -1,13 +1,21 @@
-<?xml version="1.0" ?>
+<?xml version="1.0"?>
 <!-- This does not replace URDF, and is not an extension of URDF.
   This is a format for representing semantic information about the robot structure.
-  A URDF file must exist for this robot as well, where the joints and the links that are referenced are defined -->
+  A URDF file must exist for this robot as well, where the joints and the links that are referenced
+are defined -->
 <robot xmlns:xacro="http://ros.org/wiki/xacro" name="xarm7_srdf">
-  <!-- GROUPS: Representation of a set of joints and links. This can be useful for specifying DOF to plan for, defining arms, end effectors, etc -->
-  <!-- LINKS: When a link is specified, the parent joint of that link (if it exists) is automatically included -->
-  <!-- JOINTS: When a joint is specified, the child link of that joint (which will always exist) is automatically included -->
-  <!-- CHAINS: When a chain is specified, all the links along the chain (including endpoints) are included in the group. Additionally, all the joints that are parents to included links are also included. This means that joints along the chain and the parent joint of the base link are included in the group -->
+  <!-- GROUPS: Representation of a set of joints and links. This can be useful for specifying DOF to
+  plan for, defining arms, end effectors, etc -->
+  <!-- LINKS: When a link is specified, the parent joint of that link (if it exists) is
+  automatically included -->
+  <!-- JOINTS: When a joint is specified, the child link of that joint (which will always exist) is
+  automatically included -->
+  <!-- CHAINS: When a chain is specified, all the links along the chain (including endpoints) are
+  included in the group. Additionally, all the joints that are parents to included links are also
+  included. This means that joints along the chain and the parent joint of the base link are
+  included in the group -->
   <!-- SUBGROUPS: Groups can also be formed by referencing to already defined group names -->
-  <xacro:macro name="xarm7_macro_srdf" params="prefix=''
+  <xacro:macro name="xarm7_macro_srdf"
+    params="prefix=''
     add_gripper='false' add_vacuum_gripper='false' add_other_geometry='false' ">
     <group name="${prefix}xarm7">
@@ -35,5 +43,6 @@
       </xacro:if>
     </group>
-      <!-- GROUP STATES, Purpose, Define a named state for a particular group, in terms of joint values. This is useful to define states like 'folded arms' -->
+    <!-- GROUP STATES, Purpose, Define a named state for a particular group, in terms of joint
+    values. This is useful to define states like 'folded arms' -->
     <group_state name="home" group="${prefix}xarm7">
       <joint name="${prefix}joint1" value="0.0" />
@@ -42,5 +51,5 @@
       <joint name="${prefix}joint4" value="0.0" />
       <joint name="${prefix}joint5" value="0.0" />
-           <joint name="${prefix}joint6" value="-1.5708" />
+      <joint name="${prefix}joint6" value="-1.5708" />
       <joint name="${prefix}joint7" value="0.0" />
     </group_state>
@@ -51,24 +60,15 @@
       <joint name="${prefix}joint4" value="0.0" />
       <joint name="${prefix}joint5" value="0.0" />
-           <joint name="${prefix}joint6" value="-1.5708" />
+      <joint name="${prefix}joint6" value="-1.5708" />
       <joint name="${prefix}joint7" value="0.0" />
     </group_state>
-    <group_state name="move_joint_3" group="${prefix}xarm7">
-      <joint name="${prefix}joint1" value="0.0" />
-      <joint name="${prefix}joint2" value="0.0" />
-      <joint name="${prefix}joint3" value="-1.57080" />
-      <joint name="${prefix}joint4" value="0.0" />
-      <joint name="${prefix}joint5" value="0.0" />
-           <joint name="${prefix}joint6" value="-1.5708" />
-      <joint name="${prefix}joint7" value="0.0" />
-    </group_state>
-    <group_state name="move_joint_5" group="${prefix}xarm7">
-      <joint name="${prefix}joint1" value="0.0" />
-      <joint name="${prefix}joint2" value="0.0" />
-      <joint name="${prefix}joint3" value="0.0" />
-      <joint name="${prefix}joint4" value="0.0" />
-      <joint name="${prefix}joint5" value="-1.5708" />
-           <joint name="${prefix}joint6" value="-1.5708" />
-      <joint name="${prefix}joint7" value="0.0" />
+    <group_state name="target_pose" group="${prefix}xarm7">
+      <joint name="${prefix}joint1" value="0.994838" />
+      <joint name="${prefix}joint2" value="0.174533" />
+      <joint name="${prefix}joint3" value="0.0349066" />
+      <joint name="${prefix}joint4" value="0.872665" />
+      <joint name="${prefix}joint5" value="-0.122173" />
+      <joint name="${prefix}joint6" value="-0.174533" />
+      <joint name="${prefix}joint7" value="0" />
     </group_state>
     <!-- gripper -->
@@ -92,5 +92,6 @@
       </group_state>
       <!-- END EFFECTOR, Purpose, Represent information about an end effector. -->
-      <end_effector name="${prefix}xarm_gripper" parent_link="${prefix}link_tcp" group="${prefix}xarm_gripper" />
+      <end_effector name="${prefix}xarm_gripper" parent_link="${prefix}link_tcp"
+        group="${prefix}xarm_gripper" />
       <!-- PASSIVE JOINT, Purpose, this element is used to mark joints that are not actuated -->
       <passive_joint name="${prefix}left_finger_joint" />
@@ -99,33 +100,50 @@
       <passive_joint name="${prefix}right_outer_knuckle_joint" />
       <passive_joint name="${prefix}right_finger_joint" />
-      <!-- DISABLE COLLISIONS, By default it is assumed that any link of the robot could potentially come into collision with any other link in the robot. This tag disables collision checking between a specified pair of links. -->
-      <disable_collisions link1="${prefix}left_finger" link2="${prefix}left_inner_knuckle" reason="Default" />
-      <disable_collisions link1="${prefix}left_finger" link2="${prefix}left_outer_knuckle" reason="Adjacent" />
+      <!-- DISABLE COLLISIONS, By default it is assumed that any link of the robot could potentially
+      come into collision with any other link in the robot. This tag disables collision checking
+      between a specified pair of links. -->
+      <disable_collisions link1="${prefix}left_finger" link2="${prefix}left_inner_knuckle"
+        reason="Default" />
+      <disable_collisions link1="${prefix}left_finger" link2="${prefix}left_outer_knuckle"
+        reason="Adjacent" />
       <disable_collisions link1="${prefix}left_finger" link2="${prefix}link5" reason="Never" />
       <disable_collisions link1="${prefix}left_finger" link2="${prefix}link6" reason="Never" />
       <disable_collisions link1="${prefix}left_finger" link2="${prefix}link7" reason="Never" />
       <disable_collisions link1="${prefix}left_finger" link2="${prefix}right_finger" reason="Never" />
-      <disable_collisions link1="${prefix}left_finger" link2="${prefix}right_inner_knuckle" reason="Never" />
-      <disable_collisions link1="${prefix}left_finger" link2="${prefix}right_outer_knuckle" reason="Never" />
-      <disable_collisions link1="${prefix}left_finger" link2="${prefix}xarm_gripper_base_link" reason="Never" />
-      <disable_collisions link1="${prefix}left_inner_knuckle" link2="${prefix}left_outer_knuckle" reason="Never" />
+      <disable_collisions link1="${prefix}left_finger" link2="${prefix}right_inner_knuckle"
+        reason="Never" />
+      <disable_collisions link1="${prefix}left_finger" link2="${prefix}right_outer_knuckle"
+        reason="Never" />
+      <disable_collisions link1="${prefix}left_finger" link2="${prefix}xarm_gripper_base_link"
+        reason="Never" />
+      <disable_collisions link1="${prefix}left_inner_knuckle" link2="${prefix}left_outer_knuckle"
+        reason="Never" />
       <disable_collisions link1="${prefix}left_inner_knuckle" link2="${prefix}link3" reason="Never" />
       <disable_collisions link1="${prefix}left_inner_knuckle" link2="${prefix}link5" reason="Never" />
       <disable_collisions link1="${prefix}left_inner_knuckle" link2="${prefix}link6" reason="Never" />
       <disable_collisions link1="${prefix}left_inner_knuckle" link2="${prefix}link7" reason="Never" />
-      <disable_collisions link1="${prefix}left_inner_knuckle" link2="${prefix}right_finger" reason="Never" />
-      <disable_collisions link1="${prefix}left_inner_knuckle" link2="${prefix}right_inner_knuckle" reason="Never" />
-      <disable_collisions link1="${prefix}left_inner_knuckle" link2="${prefix}right_outer_knuckle" reason="Never" />
-      <disable_collisions link1="${prefix}left_inner_knuckle" link2="${prefix}xarm_gripper_base_link" reason="Adjacent" />
+      <disable_collisions link1="${prefix}left_inner_knuckle" link2="${prefix}right_finger"
+        reason="Never" />
+      <disable_collisions link1="${prefix}left_inner_knuckle" link2="${prefix}right_inner_knuckle"
+        reason="Never" />
+      <disable_collisions link1="${prefix}left_inner_knuckle" link2="${prefix}right_outer_knuckle"
+        reason="Never" />
+      <disable_collisions link1="${prefix}left_inner_knuckle"
+        link2="${prefix}xarm_gripper_base_link" reason="Adjacent" />
       <disable_collisions link1="${prefix}left_outer_knuckle" link2="${prefix}link3" reason="Never" />
       <disable_collisions link1="${prefix}left_outer_knuckle" link2="${prefix}link6" reason="Never" />
       <disable_collisions link1="${prefix}left_outer_knuckle" link2="${prefix}link7" reason="Never" />
-      <disable_collisions link1="${prefix}left_outer_knuckle" link2="${prefix}right_finger" reason="Never" />
-      <disable_collisions link1="${prefix}left_outer_knuckle" link2="${prefix}right_inner_knuckle" reason="Never" />
-      <disable_collisions link1="${prefix}left_outer_knuckle" link2="${prefix}right_outer_knuckle" reason="Never" />
-      <disable_collisions link1="${prefix}left_outer_knuckle" link2="${prefix}xarm_gripper_base_link" reason="Adjacent" />
+      <disable_collisions link1="${prefix}left_outer_knuckle" link2="${prefix}right_finger"
+        reason="Never" />
+      <disable_collisions link1="${prefix}left_outer_knuckle" link2="${prefix}right_inner_knuckle"
+        reason="Never" />
+      <disable_collisions link1="${prefix}left_outer_knuckle" link2="${prefix}right_outer_knuckle"
+        reason="Never" />
+      <disable_collisions link1="${prefix}left_outer_knuckle"
+        link2="${prefix}xarm_gripper_base_link" reason="Adjacent" />
       <disable_collisions link1="${prefix}link3" link2="${prefix}right_inner_knuckle" reason="Never" />
       <disable_collisions link1="${prefix}link3" link2="${prefix}right_outer_knuckle" reason="Never" />
-      <disable_collisions link1="${prefix}link3" link2="${prefix}xarm_gripper_base_link" reason="Never" />
+      <disable_collisions link1="${prefix}link3" link2="${prefix}xarm_gripper_base_link"
+        reason="Never" />
       <disable_collisions link1="${prefix}link5" link2="${prefix}right_finger" reason="Never" />
       <disable_collisions link1="${prefix}link5" link2="${prefix}right_inner_knuckle" reason="Never" />
@@ -134,22 +152,35 @@
       <disable_collisions link1="${prefix}link6" link2="${prefix}right_inner_knuckle" reason="Never" />
       <disable_collisions link1="${prefix}link6" link2="${prefix}right_outer_knuckle" reason="Never" />
-      <disable_collisions link1="${prefix}link6" link2="${prefix}xarm_gripper_base_link" reason="Never" />
+      <disable_collisions link1="${prefix}link6" link2="${prefix}xarm_gripper_base_link"
+        reason="Never" />
       <disable_collisions link1="${prefix}link7" link2="${prefix}right_finger" reason="Never" />
       <disable_collisions link1="${prefix}link7" link2="${prefix}right_inner_knuckle" reason="Never" />
       <disable_collisions link1="${prefix}link7" link2="${prefix}right_outer_knuckle" reason="Never" />
-      <disable_collisions link1="${prefix}link7" link2="${prefix}xarm_gripper_base_link" reason="Adjacent" />
-      <disable_collisions link1="${prefix}right_finger" link2="${prefix}right_inner_knuckle" reason="Default" />
-      <disable_collisions link1="${prefix}right_finger" link2="${prefix}right_outer_knuckle" reason="Adjacent" />
-      <disable_collisions link1="${prefix}right_finger" link2="${prefix}xarm_gripper_base_link" reason="Never" />
-      <disable_collisions link1="${prefix}right_inner_knuckle" link2="${prefix}right_outer_knuckle" reason="Never" />
-      <disable_collisions link1="${prefix}right_inner_knuckle" link2="${prefix}xarm_gripper_base_link" reason="Adjacent" />
-      <disable_collisions link1="${prefix}right_outer_knuckle" link2="${prefix}xarm_gripper_base_link" reason="Adjacent" />
+      <disable_collisions link1="${prefix}link7" link2="${prefix}xarm_gripper_base_link"
+        reason="Adjacent" />
+      <disable_collisions link1="${prefix}right_finger" link2="${prefix}right_inner_knuckle"
+        reason="Default" />
+      <disable_collisions link1="${prefix}right_finger" link2="${prefix}right_outer_knuckle"
+        reason="Adjacent" />
+      <disable_collisions link1="${prefix}right_finger" link2="${prefix}xarm_gripper_base_link"
+        reason="Never" />
+      <disable_collisions link1="${prefix}right_inner_knuckle" link2="${prefix}right_outer_knuckle"
+        reason="Never" />
+      <disable_collisions link1="${prefix}right_inner_knuckle"
+        link2="${prefix}xarm_gripper_base_link" reason="Adjacent" />
+      <disable_collisions link1="${prefix}right_outer_knuckle"
+        link2="${prefix}xarm_gripper_base_link" reason="Adjacent" />
       <disable_collisions link1="${prefix}link_eef" link2="${prefix}left_finger" reason="Never" />
-      <disable_collisions link1="${prefix}link_eef" link2="${prefix}left_inner_knuckle" reason="Never" />
-      <disable_collisions link1="${prefix}link_eef" link2="${prefix}left_outer_knuckle" reason="Never" />
+      <disable_collisions link1="${prefix}link_eef" link2="${prefix}left_inner_knuckle"
+        reason="Never" />
+      <disable_collisions link1="${prefix}link_eef" link2="${prefix}left_outer_knuckle"
+        reason="Never" />
       <disable_collisions link1="${prefix}link_eef" link2="${prefix}right_finger" reason="Never" />
-      <disable_collisions link1="${prefix}link_eef" link2="${prefix}right_inner_knuckle" reason="Never" />
-      <disable_collisions link1="${prefix}link_eef" link2="${prefix}right_outer_knuckle" reason="Never" />
-      <disable_collisions link1="${prefix}link_eef" link2="${prefix}xarm_gripper_base_link" reason="Adjacent" />
+      <disable_collisions link1="${prefix}link_eef" link2="${prefix}right_inner_knuckle"
+        reason="Never" />
+      <disable_collisions link1="${prefix}link_eef" link2="${prefix}right_outer_knuckle"
+        reason="Never" />
+      <disable_collisions link1="${prefix}link_eef" link2="${prefix}xarm_gripper_base_link"
+        reason="Adjacent" />
     </xacro:if>
     <!-- vacuum gripper -->
@@ -158,10 +189,15 @@
         <joint name="${prefix}vacuum_gripper_fix" />
       </group> -->
-      <!-- <end_effector name="${prefix}vacuum_gripper" parent_link="${prefix}link_tcp" group="${prefix}vacuum_gripper" /> -->
+      <!-- <end_effector name="${prefix}vacuum_gripper" parent_link="${prefix}link_tcp"
+      group="${prefix}vacuum_gripper" /> -->
       <passive_joint name="${prefix}vacuum_gripper_fix" />
-      <disable_collisions link1="${prefix}link3" link2="${prefix}xarm_vacuum_gripper_link" reason="Never" />
-      <disable_collisions link1="${prefix}link6" link2="${prefix}xarm_vacuum_gripper_link" reason="Never" />
-      <disable_collisions link1="${prefix}link7" link2="${prefix}xarm_vacuum_gripper_link" reason="Adjacent" />
-      <disable_collisions link1="${prefix}link_eef" link2="${prefix}xarm_vacuum_gripper_link" reason="Adjacent" />
+      <disable_collisions link1="${prefix}link3" link2="${prefix}xarm_vacuum_gripper_link"
+        reason="Never" />
+      <disable_collisions link1="${prefix}link6" link2="${prefix}xarm_vacuum_gripper_link"
+        reason="Never" />
+      <disable_collisions link1="${prefix}link7" link2="${prefix}xarm_vacuum_gripper_link"
+        reason="Adjacent" />
+      <disable_collisions link1="${prefix}link_eef" link2="${prefix}xarm_vacuum_gripper_link"
+        reason="Adjacent" />
     </xacro:if>
     <!-- other box -->
@@ -170,10 +206,13 @@
         <joint name="${prefix}other_geometry_fix" />
       </group> -->
-      <!-- <end_effector name="${prefix}other_geometry" parent_link="${prefix}link_tcp" group="${prefix}other_geometry" /> -->
+      <!-- <end_effector name="${prefix}other_geometry" parent_link="${prefix}link_tcp"
+      group="${prefix}other_geometry" /> -->
       <passive_joint name="${prefix}other_geometry_fix" />
       <disable_collisions link1="${prefix}link3" link2="${prefix}other_geometry_link" reason="Never" />
       <disable_collisions link1="${prefix}link6" link2="${prefix}other_geometry_link" reason="Never" />
-      <disable_collisions link1="${prefix}link7" link2="${prefix}other_geometry_link" reason="Adjacent" />
-      <disable_collisions link1="${prefix}link_eef" link2="${prefix}other_geometry_link" reason="Adjacent" />
+      <disable_collisions link1="${prefix}link7" link2="${prefix}other_geometry_link"
+        reason="Adjacent" />
+      <disable_collisions link1="${prefix}link_eef" link2="${prefix}other_geometry_link"
+        reason="Adjacent" />
     </xacro:if>
     <disable_collisions link1="${prefix}link1" link2="${prefix}link2" reason="Adjacent" />

Commit message: adjustated table plane link to 0mm from base_link

File: xarm_description/urdf/xarm7/xarm7.urdf.xacro (robot description, xacro)
@@ -48,5 +48,5 @@
     </link>
     <joint name="${prefix}link_base_table_plane_joint" type="fixed">
-      <origin xyz="0.6 -0.6 -0.02" rpy="0.0 0.0 1.5708"/>
+      <origin xyz="0.6 -0.6 0.00" rpy="0.0 0.0 1.5708"/>
       <parent link="world"/>
       <child link="${prefix}table_plane"/>

File: xarm_moveit_config/srdf/_xarm7_macro.srdf.xacro (robot description, xacro)
@@ -216,4 +216,6 @@
         reason="Adjacent" />
     </xacro:if>
+    <disable_collisions link1="${prefix}table_plane" link2="${prefix}link_base" reason="Adjacent"/>
+    <disable_collisions link1="${prefix}table_plane" link2="${prefix}link1" reason="Never"/>
     <disable_collisions link1="${prefix}link1" link2="${prefix}link2" reason="Adjacent" />
     <disable_collisions link1="${prefix}link1" link2="${prefix}link3" reason="Never" />

Commit message: updated task_node to include  methods to plan with constraints

File: xarm_description/urdf/xarm7/xarm7.urdf.xacro (robot description, xacro)
@@ -144,6 +144,6 @@
       <!-- if on simulation yaw = 1.5706 -->
       <xacro:unless value = "${robot_ip == '192.1.168.225'}">
-        <!-- <origin xyz="0 0 0" rpy="1.5708 1.5708 0" /> -->
-        <xacro:common_joint_origin joint_kinematic_params="${kinematics_params['joint6']}" />
+        <origin xyz="0 0 0" rpy="1.5708 1.5708 0" />
+        <!-- <xacro:common_joint_origin joint_kinematic_params="${kinematics_params['joint6']}" /> -->
       </xacro:unless>
       <parent link="${prefix}link5" />

Commit message: added packages required by function to save data in a csv file

File: xarm_description/urdf/xarm7/xarm7.urdf.xacro (robot description, xacro)
@@ -11,4 +11,10 @@
       <xacro:property name="end_tool_collision_filename" value="end_tool/collision/end_tool"/>
     </xacro:unless>
+    <material name="Wood">
+      <color rgba="0.55 0.27 0.07 1.0"/>
+    </material>
+    <material name="Wall">
+      <color rgba="0.98 0.97 0.95 1.0"/>
+    </material>
     <!-- load params and define property -->
     <xacro:property name="default_inertial_params_filename" value="xarm7_type7_HT_BR2"/>
@@ -34,9 +40,6 @@
         <geometry>
           <mesh filename="package://xarm_description/meshes/xarm7/visual/table_plane.stl" scale="0.0001 0.0001 0.0005"/>
-          <material name="Wood">
-            <color rgba="0.219 0.445 0.286 1.0"/>
-          <texture filename=""/>
-        </material>
-        </geometry>
+        </geometry>
+        <material name="Wood"/>
       </visual>
       <collision>
@@ -47,8 +50,48 @@
       </collision>
     </link>
+    <link name="${prefix}wall_plane_1">
+      <visual>
+        <origin xyz="0.0 0.0 0.0" rpy="0.0 0.0 0.0"/>
+        <geometry>
+          <mesh filename="package://xarm_description/meshes/xarm7/visual/table_plane.stl" scale="0.0001 0.0001 0.0005"/>
+        </geometry>
+        <material name="Wall"/>
+      </visual>
+      <collision>
+        <origin xyz="0.0 0.0 0.0" rpy="0.0 0.0 0.0"/>
+        <geometry>
+          <mesh filename="package://xarm_description/meshes/xarm7/visual/table_plane.stl" scale="0.0001 0.0001 0.0005"/>
+        </geometry>
+      </collision>
+    </link>
+    <link name="${prefix}wall_plane_2">
+      <visual>
+        <origin xyz="0.0 0.0 0.0" rpy="0.0 0.0 0.0"/>
+        <geometry>
+          <mesh filename="package://xarm_description/meshes/xarm7/visual/table_plane.stl" scale="0.0001 0.0001 0.0005"/>
+        </geometry>
+        <material name="Wall"/>
+      </visual>
+      <collision>
+        <origin xyz="0.0 0.0 0.0" rpy="0.0 0.0 0.0"/>
+        <geometry>
+          <mesh filename="package://xarm_description/meshes/xarm7/visual/table_plane.stl" scale="0.0001 0.0001 0.0005"/>
+        </geometry>
+      </collision>
+    </link>
     <joint name="${prefix}link_base_table_plane_joint" type="fixed">
-      <origin xyz="0.6 -0.6 0.00" rpy="0.0 0.0 1.5708"/>
+      <origin xyz="0.6 -0.6 -0.01" rpy="0.0 0.0 1.5708"/>
       <parent link="world"/>
       <child link="${prefix}table_plane"/>
+    </joint>
+    <joint name="${prefix}link_base_wall_plane_1_joint" type="fixed">
+      <origin xyz="-0.3 -0.6 0.00" rpy="1.5708 0.0 1.5708"/>
+      <parent link="world"/>
+      <child link="${prefix}wall_plane_1"/>
+    </joint>
+    <joint name="${prefix}link_base_wall_plane_2_joint" type="fixed">
+      <origin xyz="-0.3 -0.6 0.6" rpy="1.5708 0.0 1.5708"/>
+      <parent link="world"/>
+      <child link="${prefix}wall_plane_2"/>
     </joint>
     <link name="${prefix}link_base">
