Commit message: Added instructions on how to use the bash scripts to run the simulated and the real xarm7

File: xarm_description/urdf/xarm7/xarm7.urdf.xacro (robot description, xacro)
@@ -91,5 +91,5 @@
     </joint>
     <joint name="${prefix}link_base_wall_plane_2_joint" type="fixed">
-      <origin xyz="-0.3 -0.6 0.6" rpy="1.5708 0.0 1.5708"/>
+      <origin xyz="-0.3 -0.6 0.705" rpy="1.5708 0.0 1.5708"/>
       <parent link="world"/>
       <child link="${prefix}wall_plane_2"/>
@@ -187,6 +187,6 @@
       <!-- if on simulation yaw = 1.5706 -->
       <xacro:unless value = "${robot_ip == '192.1.168.225'}">
-        <origin xyz="0 0 0" rpy="1.5708 1.5708 0" />
-        <!-- <xacro:common_joint_origin joint_kinematic_params="${kinematics_params['joint6']}" /> -->
+        <!-- <origin xyz="0 0 0" rpy="1.5708 1.5708 0" /> -->
+        <xacro:common_joint_origin joint_kinematic_params="${kinematics_params['joint6']}" />
       </xacro:unless>
       <parent link="${prefix}link5" />

Commit message: feat: add is_sim configuration to launch files and URDFs for simulation support

File: xarm_description/urdf/xarm7/xarm7.urdf.xacro (robot description, xacro)
@@ -52,4 +52,72 @@
     </xacro:unless>
     <xacro:property name="kinematics_params" value="${kinematics_config['kinematics']}"/>
+    <material name="Wood">
+      <color rgba="0.55 0.27 0.07 1.0"/>
+    </material>
+    <material name="Wall">
+      <color rgba="0.98 0.97 0.95 1.0"/>
+    </material>
+        <!-- Table plane to assist in collision detection and thus in trajectory generation  -->
+    <link name="${prefix}table_plane">
+      <visual>
+        <origin xyz="0.0 0.0 0.0" rpy="0.0 0.0 0.0"/>
+        <geometry>
+          <box size="1.0 2.0 0.015"/>
+        </geometry>
+        <material name="Wood"/>
+      </visual>
+      <collision>
+        <origin xyz="0.0 0.0 0.0" rpy="0.0 0.0 0.0"/>
+        <geometry>
+          <box size="1.0 2.0 0.015"/>
+        </geometry>
+      </collision>
+    </link>
+    <link name="${prefix}wall_plane_1">
+      <visual>
+        <origin xyz="0.0 0.0 0.0" rpy="0.0 0.0 0.0"/>
+        <geometry>
+          <box size="1.0 2.0 0.015"/>
+        </geometry>
+        <material name="Wall"/>
+      </visual>
+      <collision>
+        <origin xyz="0.0 0.0 0.0" rpy="0.0 0.0 0.0"/>
+        <geometry>
+          <box size="1.0 2.0 0.015"/>
+        </geometry>
+      </collision>
+    </link>
+    <link name="${prefix}wall_plane_2">
+      <visual>
+        <origin xyz="0.0 0.0 0.0" rpy="0.0 0.0 0.0"/>
+        <geometry>
+          <box size="1.0 2.0 0.015"/>
+        </geometry>
+        <material name="Wall"/>
+      </visual>
+      <collision>
+        <origin xyz="0.0 0.0 0.0" rpy="0.0 0.0 0.0"/>
+        <geometry>
+          <box size="1.0 2.0 0.015"/>
+        </geometry>
+      </collision>
+    </link>
+    <joint name="${prefix}link_base_table_plane_joint" type="fixed">
+      <origin xyz="0.35 0.0 -0.015" rpy="0.0 0.0 0.0"/>
+      <parent link="world"/>
+      <child link="${prefix}table_plane"/>
+    </joint>
+    <joint name="${prefix}link_base_wall_plane_1_joint" type="fixed">
+      <!-- <origin xyz="-0.3 -0.6 0.00" rpy="1.5708 0.0 1.5708"/> -->
+      <origin xyz="-0.2 0.0 0.35" rpy="0.0 ${pi/2} 0.0"/>
+      <parent link="world"/>
+      <child link="${prefix}wall_plane_1"/>
+    </joint>
+    <joint name="${prefix}link_base_wall_plane_2_joint" type="fixed">
+      <origin xyz="0.35 0.0 0.705" rpy="0.0 0.0 0.0"/>
+      <parent link="world"/>
+      <child link="${prefix}wall_plane_2"/>
+    </joint>
     <link name="${prefix}link_base">
       <inertial>
@@ -235,5 +303,15 @@
     <joint name="${prefix}joint6" type="revolute">
       <!-- <origin xyz="0 0 0" rpy="1.5708 0 0" /> -->
-      <xacro:common_joint_origin joint_kinematic_params="${kinematics_params['joint6']}" />
+      <!-- <xacro:common_joint_origin joint_kinematic_params="${kinematics_params['joint6']}" /> -->
+      <!-- If on hardware yaw = 0 -->
+      <xacro:if value = "${is_sim}">
+        <origin xyz="0 0 0" rpy="1.5708 1.5708 0" />
+        <!-- <xacro:common_joint_origin joint_kinematic_params="${kinematics_params['joint6']}" /> -->
+      </xacro:if>
+      <!-- if on simulation yaw = 1.5706 -->
+      <xacro:unless value = "${is_sim}">
+        <!-- <origin xyz="0 0 0" rpy="1.5708 1.5708 0" /> -->
+        <xacro:common_joint_origin joint_kinematic_params="${kinematics_params['joint6']}" />
+      </xacro:unless>
       <parent link="${prefix}link5" />
       <child link="${prefix}link6" />

File: xarm_description/urdf/xarm_device.urdf.xacro (robot description, xacro)
@@ -59,4 +59,6 @@
     baud_checkset="$(arg baud_checkset)" default_gripper_baud="$(arg default_gripper_baud)"
     model1300="$(arg model1300)" attach_to="$(arg attach_to)" attach_xyz="$(arg attach_xyz)" attach_rpy="$(arg attach_rpy)"
-    robot_sn="$(arg robot_sn)" use_gazebo_camera="$(arg use_gazebo_camera)" mesh_suffix="$(arg mesh_suffix)" kinematics_suffix="$(arg kinematics_suffix)" />
+    robot_sn="$(arg robot_sn)" use_gazebo_camera="$(arg use_gazebo_camera)" mesh_suffix="$(arg mesh_suffix)" kinematics_suffix="$(arg kinematics_suffix)"
+    is_sim="$(arg is_sim)"
+    />
 </robot>

File: xarm_description/urdf/xarm_device_macro.xacro (robot description, xacro)
@@ -42,4 +42,5 @@
     mesh_suffix:='stl'
     kinematics_suffix:=''
+    is_sim:=false
     "
     >

Commit message: feat: comment out 'is_sim' configuration in multiple launch files and URDF/XACRO files

File: xarm_description/urdf/xarm7/xarm7.urdf.xacro (robot description, xacro)
@@ -305,13 +305,13 @@
       <!-- <xacro:common_joint_origin joint_kinematic_params="${kinematics_params['joint6']}" /> -->
       <!-- If on hardware yaw = 0 -->
-      <xacro:if value = "${is_sim}">
-        <origin xyz="0 0 0" rpy="1.5708 1.5708 0" />
+      <!-- <xacro:if value = "${is_sim}"> -->
+        <!-- <origin xyz="0 0 0" rpy="1.5708 1.5708 0" /> -->
         <!-- <xacro:common_joint_origin joint_kinematic_params="${kinematics_params['joint6']}" /> -->
-      </xacro:if>
+      <!-- </xacro:if> -->
       <!-- if on simulation yaw = 1.5706 -->
-      <xacro:unless value = "${is_sim}">
+      <!-- <xacro:unless value = "${is_sim}"> -->
         <!-- <origin xyz="0 0 0" rpy="1.5708 1.5708 0" /> -->
         <xacro:common_joint_origin joint_kinematic_params="${kinematics_params['joint6']}" />
-      </xacro:unless>
+      <!-- </xacro:unless> -->
       <parent link="${prefix}link5" />
       <child link="${prefix}link6" />

File: xarm_description/urdf/xarm_device.urdf.xacro (robot description, xacro)
@@ -60,5 +60,4 @@
     model1300="$(arg model1300)" attach_to="$(arg attach_to)" attach_xyz="$(arg attach_xyz)" attach_rpy="$(arg attach_rpy)"
     robot_sn="$(arg robot_sn)" use_gazebo_camera="$(arg use_gazebo_camera)" mesh_suffix="$(arg mesh_suffix)" kinematics_suffix="$(arg kinematics_suffix)"
-    is_sim="$(arg is_sim)"
     />
 </robot>

File: xarm_description/urdf/xarm_device_macro.xacro (robot description, xacro)
@@ -42,5 +42,4 @@
     mesh_suffix:='stl'
     kinematics_suffix:=''
-    is_sim:=false
     "
     >

File: xarm_moveit_config/srdf/_xarm7_macro.srdf.xacro (robot description, xacro)
@@ -10,5 +10,5 @@
   <!-- SUBGROUPS: Groups can also be formed by referencing to already defined group names -->
   <xacro:macro name="xarm7_macro_srdf" params="prefix=''
-    add_gripper='false' add_vacuum_gripper='false' add_bio_gripper='false' add_other_geometry='false' is_sim='false'">
+    add_gripper='false' add_vacuum_gripper='false' add_bio_gripper='false' add_other_geometry='false'">
     <group name="${prefix}xarm7">
       <joint name="${prefix}world_joint" />

File: xarm_moveit_config/srdf/xarm.srdf.xacro (robot description, xacro)
@@ -9,7 +9,7 @@
   <xacro:arg name="add_bio_gripper" default="false" />
   <xacro:arg name="add_other_geometry" default="false" />
-  <xacro:arg name="is_sim" default="false" />
+  <!-- <xacro:arg name="is_sim" default="false" /> -->
   <xacro:include filename="$(find xarm_moveit_config)/srdf/xarm_macro.srdf.xacro" />
   <xacro:xarm_macro_srdf prefix="$(arg prefix)" dof="$(arg dof)" robot_type="$(arg robot_type)"
-    add_gripper="$(arg add_gripper)" add_vacuum_gripper="$(arg add_vacuum_gripper)" add_bio_gripper="$(arg add_bio_gripper)" add_other_geometry="$(arg add_other_geometry)" is_sim="$(arg is_sim)" />
+    add_gripper="$(arg add_gripper)" add_vacuum_gripper="$(arg add_vacuum_gripper)" add_bio_gripper="$(arg add_bio_gripper)" add_other_geometry="$(arg add_other_geometry)" />
 </robot>

File: xarm_moveit_config/srdf/xarm_macro.srdf.xacro (robot description, xacro)
@@ -2,5 +2,5 @@
 <robot xmlns:xacro="http://wiki.ros.org/xacro" name="xarm_srdf">
   <xacro:macro name="xarm_macro_srdf" params="prefix:='' dof:=7 robot_type:='xarm'
-    add_gripper:='false' add_vacuum_gripper:='false' add_bio_gripper:='false' add_other_geometry:='false' is_sim:='false'">
+    add_gripper:='false' add_vacuum_gripper:='false' add_bio_gripper:='false' add_other_geometry:='false' ">
     <xacro:if value="${dof == 5}">
       <xacro:include filename="$(find xarm_moveit_config)/srdf/_xarm5_macro.srdf.xacro" />

Commit message: fix: update joint3 limits in xarm7 URDF to correct values

File: xarm_description/urdf/xarm7/xarm7.urdf.xacro (robot description, xacro)
@@ -220,10 +220,12 @@
       <child link="${prefix}link3" />
       <axis xyz="0 0 1" />
-      <limit
+      <!-- <limit
         lower="${joint3_lower_limit}"
         upper="${joint3_upper_limit}"
         effort="30"
         velocity="3.14" />
+        -->
       <dynamics damping="5" friction="1" />
+      <limit lower="${-0.035}" upper="${0.035}" effort="30" velocity="3.14" />
     </joint>
     <link name="${prefix}link4">
