Commit message: added xarm group states

File: xarm_moveit_config/srdf/_xarm7_macro.srdf.xacro (robot description, xacro)
@@ -1,3 +1,3 @@
-<?xml version="1.0" ?>
+<?xml version="1.0.0" ?>
 <!-- This does not replace URDF, and is not an extension of URDF.
   This is a format for representing semantic information about the robot structure.
@@ -37,20 +37,38 @@
       <!-- GROUP STATES, Purpose, Define a named state for a particular group, in terms of joint values. This is useful to define states like 'folded arms' -->
     <group_state name="home" group="${prefix}xarm7">
-      <joint name="${prefix}joint1" value="0" />
-      <joint name="${prefix}joint2" value="0" />
-      <joint name="${prefix}joint3" value="0" />
-      <joint name="${prefix}joint4" value="0" />
-      <joint name="${prefix}joint5" value="0" />
-      <joint name="${prefix}joint6" value="0" />
-      <joint name="${prefix}joint7" value="0" />
+      <joint name="${prefix}joint1" value="0.0" />
+      <joint name="${prefix}joint2" value="0.0" />
+      <joint name="${prefix}joint3" value="0.0" />
+      <joint name="${prefix}joint4" value="0.0" />
+      <joint name="${prefix}joint5" value="0.0" />
+      <joint name="${prefix}joint6" value="-1.5708" />
+      <joint name="${prefix}joint7" value="0.0" />
     </group_state>
-    <group_state name="hold-up" group="${prefix}xarm7">
-      <joint name="${prefix}joint1" value="0" />
-      <joint name="${prefix}joint2" value="0" />
-      <joint name="${prefix}joint3" value="0" />
-      <joint name="${prefix}joint4" value="0" />
-      <joint name="${prefix}joint5" value="0" />
+    <group_state name="move_joint_1" group="${prefix}xarm7">
+      <joint name="${prefix}joint1" value="1.5708" />
+      <joint name="${prefix}joint2" value="0.0" />
+      <joint name="${prefix}joint3" value="0.0" />
+      <joint name="${prefix}joint4" value="0.0" />
+      <joint name="${prefix}joint5" value="0.0" />
       <joint name="${prefix}joint6" value="-1.5708" />
-      <joint name="${prefix}joint7" value="0" />
+      <joint name="${prefix}joint7" value="0.0" />
+    </group_state>
+    <group_state name="move_joint_3" group="${prefix}xarm7">
+      <joint name="${prefix}joint1" value="0.0" />
+      <joint name="${prefix}joint2" value="0.0" />
+      <joint name="${prefix}joint3" value="-1.57080" />
+      <joint name="${prefix}joint4" value="0.0" />
+      <joint name="${prefix}joint5" value="0.0" />
+      <joint name="${prefix}joint6" value="-1.5708" />
+      <joint name="${prefix}joint7" value="0.0" />
+    </group_state>
+    <group_state name="move_joint_5" group="${prefix}xarm7">
+      <joint name="${prefix}joint1" value="0.0" />
+      <joint name="${prefix}joint2" value="0.0" />
+      <joint name="${prefix}joint3" value="0.0" />
+      <joint name="${prefix}joint4" value="0.0" />
+      <joint name="${prefix}joint5" value="-1.5708" />
+      <joint name="${prefix}joint6" value="-1.5708" />
+      <joint name="${prefix}joint7" value="0.0" />
     </group_state>
     <!-- gripper -->
@@ -68,8 +86,8 @@
       </group>
       <group_state name="open" group="${prefix}xarm_gripper">
-        <joint name="${prefix}drive_joint" value="0" />
+        <joint name="${prefix}drive_joint" value="0.0" />
       </group_state>
       <group_state name="close" group="${prefix}xarm_gripper">
-        <joint name="${prefix}drive_joint" value="0.85" />
+        <joint name="${prefix}drive_joint" value="0.0.85" />
       </group_state>
       <!-- END EFFECTOR, Purpose, Represent information about an end effector. -->

Commit message: changed the group states for xarm7 group

File: xarm_moveit_config/srdf/_xarm7_macro.srdf.xacro (robot description, xacro)
@@ -42,5 +42,5 @@
       <joint name="${prefix}joint4" value="0.0" />
       <joint name="${prefix}joint5" value="0.0" />
-      <joint name="${prefix}joint6" value="-1.5708" />
+      <joint name="${prefix}joint6" value="0.0" />
       <joint name="${prefix}joint7" value="0.0" />
     </group_state>
@@ -51,5 +51,5 @@
       <joint name="${prefix}joint4" value="0.0" />
       <joint name="${prefix}joint5" value="0.0" />
-      <joint name="${prefix}joint6" value="-1.5708" />
+      <joint name="${prefix}joint6" value="0.0" />
       <joint name="${prefix}joint7" value="0.0" />
     </group_state>
@@ -60,5 +60,5 @@
       <joint name="${prefix}joint4" value="0.0" />
       <joint name="${prefix}joint5" value="0.0" />
-      <joint name="${prefix}joint6" value="-1.5708" />
+      <joint name="${prefix}joint6" value="0.0" />
       <joint name="${prefix}joint7" value="0.0" />
     </group_state>
@@ -69,5 +69,5 @@
       <joint name="${prefix}joint4" value="0.0" />
       <joint name="${prefix}joint5" value="-1.5708" />
-      <joint name="${prefix}joint6" value="-1.5708" />
+      <joint name="${prefix}joint6" value="0.0" />
       <joint name="${prefix}joint7" value="0.0" />
     </group_state>

Commit message: changed close gripper value

File: xarm_moveit_config/srdf/_xarm7_macro.srdf.xacro (robot description, xacro)
@@ -89,5 +89,5 @@
       </group_state>
       <group_state name="close" group="${prefix}xarm_gripper">
-        <joint name="${prefix}drive_joint" value="0.0.85" />
+        <joint name="${prefix}drive_joint" value="0.85" />
       </group_state>
       <!-- END EFFECTOR, Purpose, Represent information about an end effector. -->

Commit message: feat: update joint states for 'hold-up' and 'joint_1' in xarm7 macro

File: xarm_moveit_config/srdf/_xarm7_macro.srdf.xacro (robot description, xacro)
@@ -46,9 +46,18 @@
       <joint name="${prefix}joint4" value="0" />
       <joint name="${prefix}joint5" value="0" />
-      <joint name="${prefix}joint6" value="0" />
+      <joint name="${prefix}joint6" value="-1.5708" />
       <joint name="${prefix}joint7" value="0" />
     </group_state>
     <group_state name="hold-up" group="${prefix}xarm7">
       <joint name="${prefix}joint1" value="0" />
+      <joint name="${prefix}joint2" value="0" />
+      <joint name="${prefix}joint3" value="0" />
+      <joint name="${prefix}joint4" value="0" />
+      <joint name="${prefix}joint5" value="0" />
+      <joint name="${prefix}joint6" value="-1.5708" />
+      <joint name="${prefix}joint7" value="0" />
+    </group_state>
+    <group_state name="joint_1" group="${prefix}xarm7">
+      <joint name="${prefix}joint1" value="-0.78" />
       <joint name="${prefix}joint2" value="0" />
       <joint name="${prefix}joint3" value="0" />
